File: hardware/pcb/nucleo-hat/nucleo-hat.kicad_sch (KiCad schematic)
At the start: 10 parts, among them CN11 Conn_02x35_Odd_Even, CN12 Conn_02x35_Odd_Even, J1 Barrel_Jack, U1 74HC164, U2 74HC164

Commit message: pcb: version 1 for all boards
Parts:
- removed D1: D_Schottky, symbol Device:D_Schottky
- removed J1: Barrel_Jack, symbol Connector:Barrel_Jack
- added D1: D, Diode_THT:D_DO-35_SOD27_P7.62mm_Horizontal, symbol Device:D
- added P1: USB_C_Plug_USB2.0, Connector_USB:USB_C_Receptacle_GCT_USB4125-xx-x-0190_6P_TopMnt_Horizontal, symbol Connector:USB_C_Plug_USB2.0
- added R1: 390, Resistor_THT:R_Axial_DIN0204_L3.6mm_D1.6mm_P7.62mm_Horizontal, symbol Device:R
- added R10, R11, R12, R5, R6, R7, R8, R9: R, Resistor_THT:R_Axial_DIN0204_L3.6mm_D1.6mm_P7.62mm_Horizontal, symbol Device:R
- added R2: 330, Resistor_THT:R_Axial_DIN0204_L3.6mm_D1.6mm_P7.62mm_Horizontal, symbol Device:R
- added R3, R4: 1K5, Resistor_THT:R_Axial_DIN0204_L3.6mm_D1.6mm_P7.62mm_Horizontal, symbol Device:R
- added U3: SFH617A-1, Package_DIP:DIP-4_W7.62mm, symbol Isolator:SFH617A-1
- CN11, CN12: footprint (none) -> Connector_PinHeader_2.54mm:PinHeader_2x35_P2.54mm_Vertical
- IO1: renamed from IO; footprint (none) -> Connector_PinHeader_2.54mm:PinHeader_2x08_P2.54mm_Vertical
- SEQ_COL1: renamed from SEQ_COL; footprint (none) -> Connector_PinHeader_2.54mm:PinHeader_2x08_P2.54mm_Vertical
- SEQ_ROW1: renamed from SEQ_ROW; footprint (none) -> Connector_PinHeader_2.54mm:PinHeader_2x08_P2.54mm_Vertical
- SPI1: renamed from SPI; footprint (none) -> Connector_PinHeader_2.54mm:PinHeader_1x06_P2.54mm_Vertical
- U1, U2: footprint (none) -> Package_DIP:DIP-14_W7.62mm
Connections:
- net 3.3V is gone; now on net 3.3: U1.14 (VCC), U2.14 (VCC)
- net SPI_CLK is gone; now on net PA5: SPI1.5 (Pin_5)
- net SPI_CS is gone; now on net PA4: SPI1.2 (Pin_2)
- net SPI_DI is gone; now on net PA7: SPI1.6 (Pin_6)
- net SPI_DO is gone; now on net PA6: SPI1.3 (Pin_3)
- net SPI_GND is gone; now on net GND: SPI1.4 (Pin_4)
- net SPI_VCC is gone; now on net 3.3: SPI1.1 (Pin_1)
- net SR_CLK is gone; now on net PD6: U1.8 (CP), U2.8 (CP)
- net SR_CLR is gone; now on net PD5: U1.9 (~{MR}), U2.9 (~{MR})
- net SR_DATA is gone; now on net PD7: U1.1 (DSA), U1.2 (DSB)
- net GND: now also CN11.19 (Pin_19), CN11.20 (Pin_20), CN11.22 (Pin_22), CN11.60 (Pin_60), CN11.8 (Pin_8), CN12.39 (Pin_39), CN12.63 (Pin_63), IO1.13 (Pin_13), IO1.14 (Pin_14), IO1.15 (Pin_15), IO1.16 (Pin_16), IO1.2 (Pin_2), P1.A1 (GND), P1.A12 (GND), P1.B1 (GND), P1.B12 (GND), R3.2, R4.2, U3.4
- net PC10: now also CN11.1 (Pin_1), SEQ_ROW1.11 (Pin_11); no longer SEQ_ROW1.12 (Pin_12)
- net PC11: now also CN11.2 (Pin_2), SEQ_ROW1.13 (Pin_13); no longer SEQ_ROW1.14 (Pin_14)
- net PC12: now also CN11.3 (Pin_3), SEQ_ROW1.15 (Pin_15); no longer SEQ_ROW1.16 (Pin_16)
- net PC6: now also CN12.4 (Pin_4), SEQ_ROW1.3 (Pin_3); no longer SEQ_ROW1.4 (Pin_4)
- net PC7: now also CN12.19 (Pin_19), SEQ_ROW1.5 (Pin_5); no longer SEQ_ROW1.6 (Pin_6)
- net PC8: now also CN12.2 (Pin_2), SEQ_ROW1.7 (Pin_7); no longer SEQ_ROW1.8 (Pin_8)
- net PC9: now also CN12.1 (Pin_1), SEQ_ROW1.9 (Pin_9); no longer SEQ_ROW1.10 (Pin_10)
- net 3.3: now reaches CN11.16 (Pin_16)
- net 3.3: now also IO1.1 (Pin_1), R1.2
- net PB7: now reaches CN11.21 (Pin_21)
- net PB7: now also R1.1, U3.3
- net PA0: now reaches CN11.28 (Pin_28)
- net PA0: now also IO1.7 (Pin_7)
- net PA4: now reaches CN11.32 (Pin_32)
- net PD5: now reaches CN11.41 (Pin_41)
- net PD6: now reaches CN11.43 (Pin_43)
- net PD7: now reaches CN11.45 (Pin_45)
- net PE2: now reaches CN11.46 (Pin_46)
- net PE2: now also R7.2
- net PE3: now reaches CN11.47 (Pin_47)
- net PE3: now also R8.2
- net PE4: now reaches CN11.48 (Pin_48)
- net PE4: now also R9.2
- net PE5: now reaches CN11.50 (Pin_50)
- net PE5: now also R10.2
- net PF1: now reaches CN11.51 (Pin_51)
- net PF1: now also IO1.9 (Pin_9)
- net PF0: now reaches CN11.53 (Pin_53)
- net PF0: now also IO1.10 (Pin_10)
- net E5V: now reaches CN11.6 (Pin_6)
- net E5V: now also P1.A4 (VBUS), P1.A9 (VBUS), P1.B4 (VBUS), P1.B9 (VBUS)
- net PE1: now reaches CN11.61 (Pin_61)
- net PE1: now also R6.2
- net PE6: now reaches CN11.62 (Pin_62)
- net PE6: now also R11.2
- net PA11: now reaches IO1.11 (Pin_11)
- net PA11: now also CN12.14 (Pin_14)
- net PA12: now reaches IO1.12 (Pin_12)
- net PA12: now also CN12.12 (Pin_12)
- net MIDI_IN_SRC: now reaches IO1.3 (Pin_3)
- net MIDI_IN_SRC: now also R2.1
- net MIDI_IN_GND: now reaches IO1.4 (Pin_4)
- net MIDI_IN_GND: now also D1.2 (A), U3.2
- net PB6: now reaches IO1.5 (Pin_5)
- net PB6: now also CN12.17 (Pin_17)
- net PA2: now reaches IO1.6 (Pin_6)
- net PA2: now also CN12.35 (Pin_35)
- net PG14: now reaches IO1.8 (Pin_8)
- net PG14: now also CN12.61 (Pin_61)
- net PA5: now reaches CN12.11 (Pin_11)
- net PA6: now reaches CN12.13 (Pin_13)
- net PA7: now reaches CN12.15 (Pin_15)
- net PE7: now reaches CN12.44 (Pin_44)
- net PE7: now also R12.2
- net PC5: now reaches CN12.6 (Pin_6)
- net PC5: now also SEQ_ROW1.1 (Pin_1)
- net PE0: now reaches CN12.64 (Pin_64)
- net PE0: now also R5.2
- net PC3: no longer names the net of SEQ_ROW1.2 (Pin_2)
- net PC3: now also R5.1
- new net: R10.1, SEQ_ROW1.12 (Pin_12)
- new net: P1.A5 (CC), R3.1
- new net: P1.B5 (VCONN), R4.1
- new net: R7.1, SEQ_ROW1.6 (Pin_6)
- new net: D1.1 (K), R2.2, U3.1
- new net: R6.1, SEQ_ROW1.4 (Pin_4)
- new net: R9.1, SEQ_ROW1.10 (Pin_10)
- new net: R11.1, SEQ_ROW1.14 (Pin_14)
- new net: R12.1, SEQ_ROW1.16 (Pin_16)
- new net: R8.1, SEQ_ROW1.8 (Pin_8)
Other:
- moved on the sheet: IO1, SEQ_COL1, SEQ_ROW1, SPI1, U1, U2
