File: hardware/pcb/nucleo-hat/nucleo-hat.kicad_pcb (KiCad board)
At the start: 2 copper layers, 67.7 x 90.5 mm, 25 parts, among them CN11 Conn_02x35_Odd_Even, CN12 Conn_02x35_Odd_Even, P1 USB_C_Plug_USB2.0, U3 SFH617A-1

Commit message: nucleo-hat: make updates after getting board
Parts:
- moved IO1 0.86 mm to (97.9, 125.5)
Routing:
- net GND: track 163.1 -> 157.5 mm
- net PF0: track 53.6 -> 52.7 mm
- net MIDI_IN_GND: track 33.1 -> 32.3 mm
- net PF1: track 65.8 -> 64.9 mm
- net PA0: track 81.4 -> 80.6 mm
- net PG14: track 17.1 -> 18.0 mm
- net MIDI_IN_SRC: track 22.5 -> 21.7 mm
- net 3.3: track 116.4 -> 115.5 mm
- net PB6: track 70.6 -> 71.1 mm
Changed lines of the file:
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@@
 	(footprint "Connector_PinHeader_2.54mm:PinHeader_2x08_P2.54mm_Vertical"
 		(layer "F.Cu")
-		(at 98.72 125.54 90)
+		(at 97.86 125.525 90)
 		(descr "Through hole straight pin header, 2x08, 2.54mm pitch, double rows")
 		(tags "Through hole pin header THT 2x08 2.54mm double row")
@@
 	)
 	(gr_line
+		(start 117.25 61)
+		(end 117.25 128.5)
+		(stroke
+			(width 0.1)
+			(type default)
+		)
+		(layer "User.4")
+	)
+	(gr_line
 		(start 92.75 58.25)
 		(end 97.75 58.25)
@@
 	)
 	(segment
-		(start 94.75 119.03)
-		(end 98.72 123)
-		(width 0.2)
-		(layer "B.Cu")
-		(net 7)
-	)
-	(segment
 		(start 94.75 117.25)
 		(end 94.75 119.03)
@@
 	(segment
 		(start 91.415628 129.5)
-		(end 102.38 129.5)
+		(end 99 129.5)
 		(width 0.2)
 		(layer "B.Cu")
@@
 	)
 	(segment
-		(start 66.75 82)
-		(end 83.25 98.5)
+		(start 101.505 129.5)
+		(end 99 129.5)
 		(width 0.2)
 		(layer "B.Cu")
@@
 	)
 	(segment
-		(start 102.38 129.5)
-		(end 106.34 125.54)
+		(start 66.75 82)
+		(end 83.25 98.5)
 		(width 0.2)
 		(layer "B.Cu")
@@
 	)
 	(segment
+		(start 105.48 125.525)
+		(end 101.505 129.5)
+		(width 0.2)
+		(layer "B.Cu")
+		(net 19)
+	)
+	(segment
 		(start 83.25 98.5)
 		(end 83.25 121.334372)
@@
 	)
 	(segment
+		(start 103.25 129.901)
+		(end 85.365372 129.901)
+		(width 0.2)
+		(layer "B.Cu")
+		(net 44)
+	)
+	(segment
 		(start 78.628 112.128)
 		(end 74.5 108)
@@
 	)
 	(segment
-		(start 104.519 129.901)
-		(end 85.365372 129.901)
+		(start 108.02 125.525)
+		(end 103.644 129.901)
 		(width 0.2)
 		(layer "B.Cu")
@@
 	)
 	(segment
-		(start 108.88 125.54)
-		(end 104.519 129.901)
+		(start 103.644 129.901)
+		(end 103.25 129.901)
 		(width 0.2)
 		(layer "B.Cu")
@@
 	)
 	(segment
-		(start 90.04 125.54)
-		(end 98.72 125.54)
+		(start 90.055 125.525)
+		(end 90.04 125.54)
+		(width 0.2)
+		(layer "B.Cu")
+		(net 59)
+	)
+	(segment
+		(start 97.86 125.525)
+		(end 90.055 125.525)
 		(width 0.2)
 		(layer "B.Cu")
@@
 	)
 	(segment
-		(start 108.88 123)
-		(end 96.38 110.5)
+		(start 95 110.5)
+		(end 94 110.5)
 		(width 0.2)
 		(layer "B.Cu")
@@
 	)
 	(segment
-		(start 96.38 110.5)
-		(end 94 110.5)
+		(start 95.535 110.5)
+		(end 95 110.5)
 		(width 0.2)
 		(layer "B.Cu")
@@
 	)
 	(segment
-		(start 110 119.34)
-		(end 121.96 119.34)
+		(start 108.02 122.985)
+		(end 95.535 110.5)
+		(width 0.2)
+		(layer "B.Cu")
+		(net 61)
+	)
+	(segment
+		(start 121.96 119.34)
+		(end 109.125 119.34)
 		(width 0.2)
 		(layer "F.Cu")
@@
 	)
 	(segment
-		(start 106.34 123)
-		(end 110 119.34)
+		(start 109.125 119.34)
+		(end 105.48 122.985)
 		(width 0.2)
 		(layer "F.Cu")
@@
 	)
 	(segment
-		(start 112.571 89.179)
-		(end 112.571 124.389)
+		(start 111.711 90.039)
+		(end 115.5 86.25)
 		(width 0.2)
 		(layer "B.Cu")
@@
 	)
 	(segment
-		(start 112.571 124.389)
-		(end 111.42 125.54)
+		(start 111.711 124.374)
+		(end 111.711 90.039)
 		(width 0.2)
 		(layer "B.Cu")
@@
 	)
 	(segment
-		(start 115.5 86.25)
-		(end 112.571 89.179)
+		(start 110.56 125.525)
+		(end 111.711 124.374)
 		(width 0.2)
 		(layer "B.Cu")
@@
 	)
 	(segment
-		(start 115.5 85.25)
-		(end 115.5 86.25)
+		(start 115.5 86.25)
+		(end 115.5 85.25)
 		(width 0.2)
 		(layer "B.Cu")
@@
 	)
 	(segment
-		(start 102.649 82.771)
-		(end 102.649 124.389)
+		(start 101.551 83.869)
+		(end 121.96 63.46)
 		(width 0.2)
 		(layer "F.Cu")
@@
 	)
 	(segment
-		(start 121.96 63.46)
-		(end 102.649 82.771)
+		(start 101.551 124.136)
+		(end 101.551 83.869)
 		(width 0.2)
 		(layer "F.Cu")
@@
 	)
 	(segment
-		(start 102.649 124.389)
-		(end 103.8 125.54)
+		(start 102.94 125.525)
+		(end 101.551 124.136)
 		(width 0.2)
 		(layer "F.Cu")
@@
 	)
 	(segment
-		(start 103.8 123)
-		(end 117.351 109.449)
+		(start 117.351 107.75)
+		(end 117.351 90.929)
 		(width 0.2)
 		(layer "F.Cu")
@@
 	)
 	(segment
-		(start 117.351 109.449)
-		(end 117.351 90.929)
+		(start 117.351 108.574)
+		(end 117.351 107.75)
 		(width 0.2)
 		(layer "F.Cu")
@@
 	)
 	(segment
+		(start 102.94 122.985)
+		(end 117.351 108.574)
+		(width 0.2)
+		(layer "F.Cu")
+		(net 108)
+	)
+	(segment
 		(start 111.5839 53.349)
 		(end 121.7929 43.14)
@@
 	)
 	(segment
-		(start 112 87.25)
-		(end 114.5 84.75)
+		(start 114.5 84.75)
+		(end 111.101 88.149)
 		(width 0.2)
 		(layer "B.Cu")
@@
 	)
 	(segment
-		(start 111.42 123)
-		(end 111.42 87.83)
+		(start 111.101 88.149)
+		(end 111.101 122.444)
 		(width 0.2)
 		(layer "B.Cu")
@@
 	)
 	(segment
-		(start 114.5 84.75)
-		(end 114.5 84.25)
+		(start 111.101 122.444)
+		(end 110.56 122.985)
 		(width 0.2)
 		(layer "B.Cu")
@@
 	)
 	(segment
-		(start 111.42 87.83)
-		(end 112 87.25)
+		(start 114.5 84.25)
+		(end 114.5 84.75)
 		(width 0.2)
 		(layer "B.Cu")
@@
 	)
 	(segment
-		(start 70.985 119.695)
-		(end 72.781 117.899)
+		(start 96.415 119)
+		(end 95.5 119)
+		(width 0.2)
+		(layer "F.Cu")
+		(net 152)
+	)
+	(segment
+		(start 100.4 122.985)
+		(end 96.415 119)
 		(width 0.2)
 		(layer "F.Cu")
@@
 	)
 	(segment
-		(start 97.26 119)
-		(end 101.26 123)
+		(start 70.985 119.695)
+		(end 72.781 117.899)
 		(width 0.2)
 		(layer "F.Cu")
@@
 	(segment
 		(start 87.75 119)
-		(end 97.26 119)
+		(end 95.5 119)
 		(width 0.2)
 		(layer "F.Cu")
@@
 	(segment
 		(start 81.381 128.501)
-		(end 98.299 128.501)
+		(end 97.25 128.501)
 		(width 0.2)
 		(layer "F.Cu")
@@
 	)
 	(segment
-		(start 98.299 128.501)
-		(end 101.26 125.54)
+		(start 97.424 128.501)
+		(end 97.25 128.501)
 		(width 0.2)
 		(layer "F.Cu")
@@
 		(width 0.2)
 		(layer "F.Cu")
+		(net 153)
+	)
+	(segment
+		(start 100.4 125.525)
+		(end 97.424 128.501)
+		(width 0.2)
+		(layer "F.Cu")
