File: hardware/pcb/sequencer/sequencer.kicad_sch (KiCad schematic)
At the start: 106 parts, among them J1 Conn_02x08_Counter_Clockwise, J2 Conn_02x08_Counter_Clockwise, SW1 SW_SPST, SW10 SW_SPST, SW11 SW_SPST, SW12 SW_SPST, SW13 SW_SPST, SW14 SW_SPST, SW15 SW_SPST, SW16 SW_SPST, SW17 SW_SPST, SW18 SW_SPST, SW19 SW_SPST, SW2 SW_SPST, SW20 SW_SPST, SW21 SW_SPST, SW22 SW_SPST, SW23 SW_SPST, SW24 SW_SPST, SW3 SW_SPST, SW4 SW_SPST, SW5 SW_SPST, SW6 SW_SPST, SW7 SW_SPST, SW8 SW_SPST, SW9 SW_SPST

Commit message: sequencer: update pcb layout
Parts:
- removed J1, J2: Conn_02x08_Counter_Clockwise, Connector_PinHeader_1.27mm:PinHeader_2x08_P1.27mm_Vertical, symbol Connector_Generic:Conn_02x08_Counter_Clockwise
- removed R17, R18, R19, R20, R21, R22, R23, R24, R25, R26, R27, R28, R29, R30, R31, R32: R, Resistor_SMD:R_0201_0603Metric, symbol Device:R
- added J1, J2: Conn_02x08_Odd_Even, Connector_PinHeader_1.27mm:PinHeader_2x08_P1.27mm_Vertical, symbol Connector_Generic:Conn_02x08_Odd_Even
- renumbered R13 to S1, R6 to S10, R7 to S11, R8 to S12, R1 to S13, R2 to S14, R3 to S15, R4 to S16, R14 to S2, R15 to S3, R16 to S4, R9 to S5, R10 to S6, R11 to S7, R12 to S8, R5 to S9
Connections:
- net I1: now also J1.1 (Pin_1)
- net I10: now also J1.4 (Pin_4)
- net I11: now also J1.6 (Pin_6)
- net I12: now also J1.8 (Pin_8)
- net I13: now also J1.10 (Pin_10)
- net I14: now also J1.12 (Pin_12)
- net I15: now also J1.14 (Pin_14)
- net I16: now also J1.16 (Pin_16)
- net I2: now also J1.3 (Pin_3)
- net I3: now also J1.5 (Pin_5)
- net I4: now also J1.7 (Pin_7)
- net I5: now also J1.9 (Pin_9)
- net I6: now also J1.11 (Pin_11)
- net I7: now also J1.13 (Pin_13)
- net I8: now also J1.15 (Pin_15)
- net I9: now also J1.2 (Pin_2)
- net O1: now also J2.1 (Pin_1)
- net O10: now also J2.4 (Pin_4)
- net O11: now also J2.6 (Pin_6)
- net O12: now also J2.8 (Pin_8)
- net O13: now also J2.10 (Pin_10)
- net O14: now also J2.12 (Pin_12)
- net O15: now also J2.14 (Pin_14)
- net O16: now also J2.16 (Pin_16)
- net O2: now also J2.3 (Pin_3)
- net O3: now also J2.5 (Pin_5)
- net O4: now also J2.7 (Pin_7)
- net O5: now also J2.9 (Pin_9)
- net O6: now also J2.11 (Pin_11)
- net O7: now also J2.13 (Pin_13)
- net O8: now also J2.15 (Pin_15)
- net O9: now also J2.2 (Pin_2)
- net C2: now reaches S10.2, S14.2, S2.2, S6.2, SW10.2 (B), SW11.2 (B), SW12.2 (B), SW7.2 (B), SW8.2 (B), SW9.2 (B)
- net C2: now also D31.2 (A), D32.2 (A), D33.2 (A), D34.2 (A), D35.2 (A), D36.2 (A)
- net C4: now reaches S12.2, S16.2, S4.2, S8.2, SW19.2 (B), SW20.2 (B), SW21.2 (B), SW22.2 (B), SW23.2 (B), SW24.2 (B)
- net C4: now also D43.2 (A), D44.2 (A), D45.2 (A), D46.2 (A), D47.2 (A), D48.2 (A)
- net C1: now reaches D25.2 (A), D26.2 (A), D27.2 (A), D28.2 (A), D29.2 (A), D30.2 (A)
- net C1: now also S1.2, S13.2, S5.2, S9.2, SW1.2 (B), SW2.2 (B), SW3.2 (B), SW4.2 (B), SW5.2 (B), SW6.2 (B)
- net C3: now reaches D37.2 (A), D42.2 (A)
- net C3: now also D38.2 (A), D39.2 (A), D40.2 (A), D41.2 (A), S11.2, S15.2, S3.2, S7.2, SW13.2 (B), SW14.2 (B), SW15.2 (B), SW16.2 (B), SW17.2 (B), SW18.2 (B)
Other:
- moved on the sheet: S1, S10, S11, S12, S13, S14, S15, S16, S2, S3, S4, S5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

Commit message: sequencer: route pcb
Parts:
- S1, S10, S11, S12, S13, S14, S15, S16, S2, S3, S4, S5, S6, S7, S8, S9: footprint Resistor_SMD:R_0201_0603Metric -> Resistor_SMD:R_0603_1608Metric
Changed lines of the file:
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@@
 			)
 		)
-		(property "Footprint" "Resistor_SMD:R_0201_0603Metric"
+		(property "Footprint" "Resistor_SMD:R_0603_1608Metric"
 			(at 140.462 30.48 90)
 			(effects
@@
 			)
 		)
-		(property "Footprint" "Resistor_SMD:R_0201_0603Metric"
+		(property "Footprint" "Resistor_SMD:R_0603_1608Metric"
 			(at 122.682 30.48 90)
 			(effects
@@
 			)
 		)
-		(property "Footprint" "Resistor_SMD:R_0201_0603Metric"
+		(property "Footprint" "Resistor_SMD:R_0603_1608Metric"
 			(at 163.322 30.48 90)
 			(effects
@@
 			)
 		)
-		(property "Footprint" "Resistor_SMD:R_0201_0603Metric"
+		(property "Footprint" "Resistor_SMD:R_0603_1608Metric"
 			(at 153.162 30.48 90)
 			(effects
@@
 			)
 		)
-		(property "Footprint" "Resistor_SMD:R_0201_0603Metric"
+		(property "Footprint" "Resistor_SMD:R_0603_1608Metric"
 			(at 176.022 30.48 90)
 			(effects
@@
 			)
 		)
-		(property "Footprint" "Resistor_SMD:R_0201_0603Metric"
+		(property "Footprint" "Resistor_SMD:R_0603_1608Metric"
 			(at 112.522 30.48 90)
 			(effects
@@
 			)
 		)
-		(property "Footprint" "Resistor_SMD:R_0201_0603Metric"
+		(property "Footprint" "Resistor_SMD:R_0603_1608Metric"
 			(at 158.242 30.48 90)
 			(effects
@@
 			)
 		)
-		(property "Footprint" "Resistor_SMD:R_0201_0603Metric"
+		(property "Footprint" "Resistor_SMD:R_0603_1608Metric"
 			(at 117.602 30.48 90)
 			(effects
@@
 			)
 		)
-		(property "Footprint" "Resistor_SMD:R_0201_0603Metric"
+		(property "Footprint" "Resistor_SMD:R_0603_1608Metric"
 			(at 181.102 30.48 90)
 			(effects
@@
 			)
 		)
-		(property "Footprint" "Resistor_SMD:R_0201_0603Metric"
+		(property "Footprint" "Resistor_SMD:R_0603_1608Metric"
 			(at 130.302 30.48 90)
 			(effects
@@
 			)
 		)
-		(property "Footprint" "Resistor_SMD:R_0201_0603Metric"
+		(property "Footprint" "Resistor_SMD:R_0603_1608Metric"
 			(at 168.402 30.48 90)
 			(effects
@@
 			)
 		)
-		(property "Footprint" "Resistor_SMD:R_0201_0603Metric"
+		(property "Footprint" "Resistor_SMD:R_0603_1608Metric"
 			(at 186.182 30.48 90)
 			(effects
@@
 			)
 		)
-		(property "Footprint" "Resistor_SMD:R_0201_0603Metric"
+		(property "Footprint" "Resistor_SMD:R_0603_1608Metric"
 			(at 135.382 30.48 90)
 			(effects
@@
 			)
 		)
-		(property "Footprint" "Resistor_SMD:R_0201_0603Metric"
+		(property "Footprint" "Resistor_SMD:R_0603_1608Metric"
 			(at 191.262 30.48 90)
 			(effects
@@
 			)
 		)
-		(property "Footprint" "Resistor_SMD:R_0201_0603Metric"
+		(property "Footprint" "Resistor_SMD:R_0603_1608Metric"
 			(at 107.442 30.48 90)
 			(effects
@@
 			)
 		)
-		(property "Footprint" "Resistor_SMD:R_0201_0603Metric"
+		(property "Footprint" "Resistor_SMD:R_0603_1608Metric"
 			(at 145.542 30.48 90)
 			(effects

Commit message: hardware: add schematics
add controls, io, keys, and nucleo hat boards
Parts:
- added J3, J4, J5, J6, J7, J8: Conn_01x01, Connector_PinHeader_1.27mm:PinHeader_1x01_P1.27mm_Vertical, symbol Connector_Generic:Conn_01x01
Connections:
- net C1: now also J3.1 (Pin_1)
- net C2: now also J4.1 (Pin_1)
- net C3: now also J5.1 (Pin_1)
- net C4: now also J6.1 (Pin_1)
- net O7: now also J7.1 (Pin_1)
- net O8: now also J8.1 (Pin_1)

Commit message: sequencer: move keys and controls to this pcb
it's just easier to do it this way
Parts:
- removed J3, J4, J5, J6, J7, J8: Conn_01x01, Connector_PinHeader_1.27mm:PinHeader_1x01_P1.27mm_Vertical, symbol Connector_Generic:Conn_01x01
- added D49, D50, D51, D52, D53, D54, D55, D56: D, Diode_THT:D_DO-35_SOD27_P7.62mm_Horizontal, symbol Device:D
- added D57, D58, D59, D60, D61, D62, D63, D64: LED, LED_SMD:LED_0805_2012Metric, symbol Device:LED
- added SW25, SW26, SW27, SW28, SW29, SW30, SW31, SW32: SW_SPST, Button_Switch_Keyboard:SW_Cherry_MX_1.00u_PCB, symbol Switch:SW_SPST
Connections:
- net C1: now also D57.2 (A), D61.2 (A), SW25.2 (B), SW29.2 (B)
- net C2: now also D58.2 (A), D62.2 (A), SW26.2 (B), SW30.2 (B)
- net C3: now also D59.2 (A), D63.2 (A), SW27.2 (B), SW31.2 (B)
- net C4: now also D60.2 (A), D64.2 (A), SW28.2 (B), SW32.2 (B)
- net O15: now also D57.1 (K), D58.1 (K), D59.1 (K), D60.1 (K)
- net O16: now also D61.1 (K), D62.1 (K), D63.1 (K), D64.1 (K)
- net O7: now also D49.1 (K), D50.1 (K), D51.1 (K), D52.1 (K)
- net O8: now also D53.1 (K), D54.1 (K), D55.1 (K), D56.1 (K)
- new net: D54.2 (A), SW30.1 (A)
- new net: D56.2 (A), SW32.1 (A)
- new net: D50.2 (A), SW26.1 (A)
- new net: D53.2 (A), SW29.1 (A)
- new net: D52.2 (A), SW28.1 (A)
- new net: D49.2 (A), SW25.1 (A)
- new net: D55.2 (A), SW31.1 (A)
- new net: D51.2 (A), SW27.1 (A)

Commit message: pcb: version 1 for all boards
Parts:
- J1, J2: footprint Connector_PinHeader_1.27mm:PinHeader_2x08_P1.27mm_Vertical -> Connector_PinHeader_2.54mm:PinHeader_2x08_P2.54mm_Vertical
Changed lines of the file:
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@@
 			)
 		)
-		(property "Footprint" "Connector_PinHeader_1.27mm:PinHeader_2x08_P1.27mm_Vertical"
+		(property "Footprint" "Connector_PinHeader_2.54mm:PinHeader_2x08_P2.54mm_Vertical"
 			(at 81.28 30.48 0)
 			(effects
@@
 			)
 		)
-		(property "Footprint" "Connector_PinHeader_1.27mm:PinHeader_2x08_P1.27mm_Vertical"
+		(property "Footprint" "Connector_PinHeader_2.54mm:PinHeader_2x08_P2.54mm_Vertical"
 			(at 46.99 30.48 0)
 			(effects

Commit message: sequencer: update front panel pcb
- switch to through hole leds
- move mounting holes to board edges
- use solder bridges for column selection
- add separate header for led driving

Signed-off-by: Emma Davenport <emma.v.davenport@gmail.com>
Parts:
- added J3: Conn_02x08_Odd_Even, Connector_PinHeader_2.54mm:PinHeader_2x08_P2.54mm_Vertical, symbol Connector_Generic:Conn_02x08_Odd_Even
- added S17, S18, S19, S20, S21, S22, S23, S24, S25, S26, S27, S28, S29, S30, S31, S32: R, Jumper:SolderJumper-2_P1.3mm_Open_RoundedPad1.0x1.5mm, symbol Device:R
- D25, D26, D27, D28, D29, D30, D31, D32, D33, D34, D35, D36, D37, D38, D39, D40, D41, D42, D43, D44, D45, D46, D47, D48, D57, D58, D59, D60, D61, D62, D63, D64: footprint LED_SMD:LED_0805_2012Metric -> LED_THT:LED_D3.0mm
- S1, S10, S11, S12, S13, S14, S15, S16, S2, S3, S4, S5, S6, S7, S8, S9: footprint Resistor_SMD:R_0603_1608Metric -> Jumper:SolderJumper-2_P1.3mm_Open_RoundedPad1.0x1.5mm
Connections:
- net C1: no longer D25.2 (A), D26.2 (A), D27.2 (A), D28.2 (A), D29.2 (A), D30.2 (A), D57.2 (A), D61.2 (A)
- net C2: no longer D31.2 (A), D32.2 (A), D33.2 (A), D34.2 (A), D35.2 (A), D36.2 (A), D58.2 (A), D62.2 (A)
- net C3: no longer D37.2 (A), D38.2 (A), D39.2 (A), D40.2 (A), D41.2 (A), D42.2 (A), D59.2 (A), D63.2 (A)
- net C4: no longer D43.2 (A), D44.2 (A), D45.2 (A), D46.2 (A), D47.2 (A), D48.2 (A), D60.2 (A), D64.2 (A)
- new net C5: D25.2 (A), D26.2 (A), D27.2 (A), D28.2 (A), D29.2 (A), D30.2 (A), D57.2 (A), D61.2 (A), S17.2, S21.2, S25.2, S29.2
- new net C6: D31.2 (A), D32.2 (A), D33.2 (A), D34.2 (A), D35.2 (A), D36.2 (A), D58.2 (A), D62.2 (A), S18.2, S22.2, S26.2, S30.2
- new net C7: D37.2 (A), D38.2 (A), D39.2 (A), D40.2 (A), D41.2 (A), D42.2 (A), D59.2 (A), D63.2 (A), S19.2, S23.2, S27.2, S31.2
- new net C8: D43.2 (A), D44.2 (A), D45.2 (A), D46.2 (A), D47.2 (A), D48.2 (A), D60.2 (A), D64.2 (A), S20.2, S24.2, S28.2, S32.2
- new net L1: J3.1 (Pin_1), S17.1
- new net L10: J3.4 (Pin_4), S26.1
- new net L11: J3.6 (Pin_6), S27.1
- new net L12: J3.8 (Pin_8), S28.1
- new net L13: J3.10 (Pin_10), S29.1
- new net L14: J3.12 (Pin_12), S30.1
- new net L15: J3.14 (Pin_14), S31.1
- new net L16: J3.16 (Pin_16), S32.1
- new net L2: J3.3 (Pin_3), S18.1
- new net L3: J3.5 (Pin_5), S19.1
- new net L4: J3.7 (Pin_7), S20.1
- new net L5: J3.9 (Pin_9), S21.1
- new net L6: J3.11 (Pin_11), S22.1
- new net L7: J3.13 (Pin_13), S23.1
- new net L8: J3.15 (Pin_15), S24.1
- new net L9: J3.2 (Pin_2), S25.1
Other:
- moved on the sheet: S1, S10, S11, S12, S13, S14, S15, S16, S2, S3, S4, S5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
