File: hardware/pcb/sequencer/sequencer.kicad_pcb (KiCad board)
At the start: 2 copper layers, 78 x 177.5 mm, 165 parts, among them J1 Conn_02x08_Odd_Even, J2 Conn_02x08_Odd_Even, J3 Conn_02x08_Odd_Even, SW1 SW_SPST, SW10 SW_SPST, SW11 SW_SPST, SW12 SW_SPST, SW13 SW_SPST, SW14 SW_SPST, SW15 SW_SPST, SW16 SW_SPST, SW17 SW_SPST, SW18 SW_SPST, SW19 SW_SPST, SW2 SW_SPST, SW20 SW_SPST, SW21 SW_SPST, SW22 SW_SPST, SW23 SW_SPST, SW24 SW_SPST, SW25 SW_SPST, SW26 SW_SPST, SW27 SW_SPST, SW28 SW_SPST, SW29 SW_SPST, SW3 SW_SPST, SW30 SW_SPST, SW31 SW_SPST, SW32 SW_SPST, SW4 SW_SPST, SW5 SW_SPST, SW6 SW_SPST, SW7 SW_SPST, SW8 SW_SPST, SW9 SW_SPST

Commit message: update pcbs
Parts:
- removed the G*** at (221.8, 163.0)
- removed the G*** at (213.2, 137.8)
- D1, D10, D11, D12, D13, D14, D15, D16, D17, D18, D19, D2, D20, D21, D22, D23, D24, D3, D4, D49, D5, D50, D51, D52, D53, D54, D55, D56, D6, D7, D8, D9: footprint Diode_THT:D_DO-35_SOD27_P7.62mm_Horizontal -> sequencer:D_DO-35_SOD27_P7.62mm_Horizontal_no_silk
- D25, D26, D27, D28, D29, D30, D31, D32, D33, D34, D35, D36, D37, D38, D39, D40, D41, D42, D43, D44, D45, D46, D47, D48, D57, D58, D59, D60, D61, D62, D63, D64: footprint LED_THT:LED_D3.0mm -> sequencer:LED_D3.0mm_no_silk
- SW1, SW10, SW11, SW12, SW13, SW14, SW15, SW16, SW17, SW18, SW19, SW2, SW20, SW21, SW22, SW23, SW24, SW25, SW26, SW27, SW28, SW29, SW3, SW30, SW31, SW32, SW4, SW5, SW6, SW7, SW8, SW9: footprint Button_Switch_Keyboard:SW_Cherry_MX_1.00u_PCB -> sequencer:SW_Cherry_MX_1.00u_PCB_no_footprint
